File: pico-w-ha-node.kicad_pcb (KiCad board)
At the start: 2 copper layers, 31 parts, among them J1 USB_C_Receptacle_PowerOnly_6P, J4 Conn_01x02, J5 Conn_01x02, J6 Conn_01x03, J7 Conn_01x03, Q1 STD18NF03L, Q2 STD18NF03L, Q3 str2n2vh5, Q9 str2n2vh5, SW1 SW_Push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

Commit message: Adds 3rd output via USB-A and some additional capacitors.
Parts:
- removed SW1: SW_Push, Button_Switch_SMD:SW_SPST_TL3305A
- added C2: 820µ, Capacitor_THT:CP_Radial_D10.0mm_P5.00mm, F.Cu at (109.2, 104.1)
- added C3: C, Capacitor_THT:CP_Radial_D10.0mm_P5.00mm, F.Cu at (126.1, 72.5)
- added C4: 100n, Capacitor_SMD:C_0603_1608Metric_Pad1.08x0.95mm_HandSolder, B.Cu at (147.5, 100.8)
- added C5: 820µ, Capacitor_THT:CP_Radial_D10.0mm_P5.00mm, F.Cu at (109.2, 85.4)
- added C6: 100n, Capacitor_SMD:C_0805_2012Metric, F.Cu at (99.8, 70.0)
- added C7: 100n, Capacitor_SMD:C_0805_2012Metric, F.Cu at (108.8, 94.8)
- added C8: 100n, Capacitor_SMD:C_0805_2012Metric, F.Cu at (156.7, 70.0)
- added C9: 820µ, Capacitor_THT:CP_Radial_D10.0mm_P5.00mm, F.Cu at (153.1, 62.8)
- added J2: Conn_01x02, Connector_Molex:Molex_Micro-Fit_3.0_43650-0212_1x02-1MP_P3.00mm_Horizontal, F.Cu at (157.3, 99.5)
- added Q4: str2n2vh5, Package_TO_SOT_SMD:SOT-23, F.Cu at (108.8, 97.8)
- added R15: 10k, Resistor_SMD:R_0603_1608Metric_Pad0.98x0.95mm_HandSolder, F.Cu at (163.6, 58.2)
- added R16: 220, Resistor_SMD:R_0603_1608Metric_Pad0.98x0.95mm_HandSolder, F.Cu at (163.6, 60.8)
- C1, R14, R5, R6, U1: moved to B.Cu
- F1: footprint Fuse:Fuse_0603_1608Metric_Pad1.05x0.95mm_HandSolder -> Fuse:Fuse_1206_3216Metric
- Q1, Q2: value STD18NF03L -> str2n2vh5; footprint Package_TO_SOT_SMD:TO-252-2 -> Package_TO_SOT_SMD:SOT-23
- moved R3 73.1 mm to (112.8, 117.3)
- moved R4 72.9 mm to (112.8, 119.0)
- moved J6 68.3 mm to (157.3, 120.5)
- moved Q2 51.1 mm to (152.1, 70.8)
- moved D1 49.0 mm to (144.4, 92.5)
- moved R9 41.3 mm to (144.4, 94.0)
- moved J5 40.4 mm to (98.1, 114.0), turned to -90 degrees
- moved F1 34.3 mm to (146.8, 86.2), turned to 180 degrees
- moved R6 29.9 mm to (156.0, 87.0)
- moved R5 26.9 mm to (156.0, 85.5)
- moved Q1 17.0 mm to (108.8, 66.0), turned to 0 degrees
- moved R1 16.6 mm to (112.8, 100.2), turned to 0 degrees
- moved R2 16.0 mm to (112.8, 98.8)
- moved J4 12.5 mm to (100.1, 97.6), turned to -90 degrees
- moved J7 7.47 mm to (91.5, 132.5)
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Connections:
- A1 pad 30: Net-(A1-RUN) -> unconnected-(A1-RUN-Pad30)
- Q1 pad 2: /LS1_OUT -> GND
- Q1 pad 3: GND -> /LS2_OUT
- Q2 pad 2: /LS2_OUT -> GND
- Q2 pad 3: GND -> /LS3_OUT
- R2 pad 1: Net-(Q1-G) -> Net-(Q4-G)
- R4 pad 1: Net-(Q2-G) -> Net-(Q1-G)
Routing:
- net Net-(J2-Pin_1): track 0.00 -> 25.8 mm
- net +3V3: track 0.00 -> 17.8 mm, vias 0 -> 1
- net +5V: track 0.00 -> 6.03 mm, vias 0 -> 4
- net /LS1_OUT: track 0.00 -> 5.34 mm
- net Net-(Q1-G): track 0.00 -> 2.61 mm
- net Net-(Q4-G): track 0.00 -> 2.15 mm
- net /LS2_EN: track 0.00 -> 1.75 mm
- net GND: track 0.00 -> 1.55 mm, vias 0 -> 2
- net Net-(J1-CC2): track 0.00 -> 1.52 mm, vias 0 -> 1
- net Net-(J1-CC1): track 0.00 -> 1.52 mm, vias 0 -> 1
- net Net-(D1-A): track 0.00 -> 1.52 mm
- net /LS1_EN: track 0.00 -> 1.50 mm
- net Net-(A1-GPIO26_ADC0): track 7.81 -> 6.96 mm, vias 0 -> 1
- added copper zone on B.Cu, net +5V
- added copper zone on F.Cu, net GND
